File: C64 Modulator.kicad_pcb (KiCad board)
At the start: 2 copper layers, 63.5 x 63.4 mm, 38 parts, among them J10 , J11 , J12 , J13 , J14 , J2 8765, J3 4321, J4 AUD_STEREO, J5 TRS_3.5mm, J6 RCA_PLUG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

Commit message: Readded D1
Parts:
- added D1: 1n4148, Diodes_THT:D_DO-35_SOD27_P7.62mm_Horizontal, F.Cu at (154.9, 90.2)
- added J7: , anchors:anchor_circle, F.Cu at (120.0, 79.4)
Connections:
- C5 pad 1: VCC -> Net-(C5-Pad1)
- C7 pad 1: VCC -> Net-(C5-Pad1)
- U1 pad 3: VCC -> Net-(C5-Pad1)
Routing:
- net Net-(C5-Pad1): track 0.00 -> 33.5 mm
- net VCC: track 86.1 -> 58.5 mm
Changed lines of the file:
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@@
 (kicad_pcb (version 4) (host pcbnew 4.0.7)
   (general
-    (links 59)
+    (links 61)
     (no_connects 0)
     (area 118.669999 62.154999 182.360001 125.745001)
@@
     (tracks 152)
     (zones 0)
-    (modules 38)
-    (nets 20)
+    (modules 40)
+    (nets 21)
   )
   (page A4)
@@
     (mod_text_size 1 1)
     (mod_text_width 0.15)
-    (pad_size 1.7 1.7)
-    (pad_drill 1)
+    (pad_size 3.19786 1.99898)
+    (pad_drill 2.1971)
     (pad_to_mask_clearance 0.2)
     (aux_axis_origin 0 0)
@@
   (net 18 "Net-(J3-Pad2)")
   (net 19 "Net-(J3-Pad3)")
+  (net 20 "Net-(C5-Pad1)")
   (net_class Default "This is the default net class."
     (clearance 0.2)
@@
     (add_net AUDIO_IN)
     (add_net COMPOSITE)
+    (add_net "Net-(C5-Pad1)")
     (add_net "Net-(J4-Pad1)")
     (add_net VCC)
@@
     (pad 2 thru_hole oval (at 3.81 -3.81 180) (size 1.99898 3.19786) (drill oval 0.99568 2.1971) (layers *.Cu *.Mask F.SilkS)
       (net 6 COMPOSITE))
-    (pad 1 thru_hole oval (at -1 -1.27 180) (size 3.19786 1.99898) (drill oval 2.1971 0.99568) (layers *.Cu *.Mask F.SilkS)
+    (pad 1 thru_hole oval (at 0 -1.27 180) (size 3.19786 1.99898) (drill oval 2.1971 0.99568) (layers *.Cu *.Mask F.SilkS)
       (net 3 GND))
     (pad 2 thru_hole oval (at -3.81 -3.81 180) (size 1.99898 3.19786) (drill oval 0.99568 2.1971) (layers *.Cu *.Mask F.SilkS)
@@
     )
     (pad 1 thru_hole rect (at 0 0) (size 1.6 1.6) (drill 0.8) (layers *.Cu *.Mask)
-      (net 7 VCC))
+      (net 20 "Net-(C5-Pad1)"))
     (pad 2 thru_hole circle (at 2.5 0) (size 1.6 1.6) (drill 0.8) (layers *.Cu *.Mask)
       (net 3 GND))
@@
     )
     (pad 1 thru_hole circle (at 0 0) (size 1.6 1.6) (drill 0.8) (layers *.Cu *.Mask)
-      (net 7 VCC))
+      (net 20 "Net-(C5-Pad1)"))
     (pad 2 thru_hole circle (at 5 0) (size 1.6 1.6) (drill 0.8) (layers *.Cu *.Mask)
       (net 3 GND))
@@
       (net 3 GND))
     (pad 3 thru_hole oval (at 5.08 0 90) (size 1.8 1.8) (drill 1) (layers *.Cu *.Mask)
-      (net 7 VCC))
+      (net 20 "Net-(C5-Pad1)"))
     (model ${KISYS3DMOD}/TO_SOT_Packages_THT.3dshapes/TO-220-3_Horizontal.wrl
       (at (xyz 0.1 0 0))
@@
     )
   )
+  (module Diodes_THT:D_DO-35_SOD27_P7.62mm_Horizontal (layer F.Cu)
+    (at 154.94 90.17 90)
+    (descr "D, DO-35_SOD27 series, Axial, Horizontal, pin pitch=7.62mm, , length*diameter=4*2mm^2, , http://www.diodes.com/_files/packages/DO-35.pdf")
+    (tags "D DO-35_SOD27 series Axial Horizontal pin pitch 7.62mm  length 4mm diameter 2mm")
+    (fp_text reference D1 (at 3.81 0 90) (layer F.SilkS)
+      (effects (font (size 1 1) (thickness 0.15)))
+    )
+    (fp_text value 1n4148 (at 3.81 2.06 90) (layer F.Fab)
+      (effects (font (size 1 1) (thickness 0.15)))
+    )
+    (fp_text user %R (at 3.81 0 90) (layer F.Fab)
+      (effects (font (size 1 1) (thickness 0.15)))
+    )
+    (fp_line (start 1.81 -1) (end 1.81 1) (layer F.Fab) (width 0.1))
+    (fp_line (start 1.81 1) (end 5.81 1) (layer F.Fab) (width 0.1))
+    (fp_line (start 5.81 1) (end 5.81 -1) (layer F.Fab) (width 0.1))
+    (fp_line (start 5.81 -1) (end 1.81 -1) (layer F.Fab) (width 0.1))
+    (fp_line (start 0 0) (end 1.81 0) (layer F.Fab) (width 0.1))
+    (fp_line (start 7.62 0) (end 5.81 0) (layer F.Fab) (width 0.1))
+    (fp_line (start 2.41 -1) (end 2.41 1) (layer F.Fab) (width 0.1))
+    (fp_line (start 1.75 -1.06) (end 1.75 1.06) (layer F.SilkS) (width 0.12))
+    (fp_line (start 1.75 1.06) (end 5.87 1.06) (layer F.SilkS) (width 0.12))
+    (fp_line (start 5.87 1.06) (end 5.87 -1.06) (layer F.SilkS) (width 0.12))
+    (fp_line (start 5.87 -1.06) (end 1.75 -1.06) (layer F.SilkS) (width 0.12))
+    (fp_line (start 0.98 0) (end 1.75 0) (layer F.SilkS) (width 0.12))
+    (fp_line (start 6.64 0) (end 5.87 0) (layer F.SilkS) (width 0.12))
+    (fp_line (start 2.41 -1.06) (end 2.41 1.06) (layer F.SilkS) (width 0.12))
+    (fp_line (start -1.05 -1.35) (end -1.05 1.35) (layer F.CrtYd) (width 0.05))
+    (fp_line (start -1.05 1.35) (end 8.7 1.35) (layer F.CrtYd) (width 0.05))
+    (fp_line (start 8.7 1.35) (end 8.7 -1.35) (layer F.CrtYd) (width 0.05))
+    (fp_line (start 8.7 -1.35) (end -1.05 -1.35) (layer F.CrtYd) (width 0.05))
+    (pad 1 thru_hole rect (at 0 0 90) (size 1.6 1.6) (drill 0.8) (layers *.Cu *.Mask)
+      (net 7 VCC))
+    (pad 2 thru_hole oval (at 7.62 0 90) (size 1.6 1.6) (drill 0.8) (layers *.Cu *.Mask)
+      (net 20 "Net-(C5-Pad1)"))
+    (model ${KISYS3DMOD}/Diodes_THT.3dshapes/D_DO-35_SOD27_P7.62mm_Horizontal.wrl
+      (at (xyz 0 0 0))
+      (scale (xyz 0.393701 0.393701 0.393701))
+      (rotate (xyz 0 0 0))
+    )
+  )
+  (module anchors:anchor_circle (layer F.Cu)
+    (at 120.015 79.375)
+    (fp_text reference J7 (at 0 1.524) (layer F.SilkS) hide
+      (effects (font (size 1 1) (thickness 0.15)))
+    )
+    (fp_text value " " (at 0 -2.54) (layer F.Fab) hide
+      (effects (font (size 1 1) (thickness 0.15)))
+    )
+    (pad 1 thru_hole circle (at 0 0.025) (size 1.524 1.524) (drill 0.762) (layers *.Cu *.Mask)
+      (net 3 GND))
+  )
   (gr_text "Revision B" (at 177.165 63.5) (layer F.SilkS)
     (effects (font (size 1 1) (thickness 0.15)))
@@
   (gr_line (start 162.56 78.74) (end 165.1 78.74) (angle 90) (layer B.SilkS) (width 0.2))
   (gr_line (start 162.56 76.835) (end 162.56 78.74) (angle 90) (layer B.SilkS) (width 0.2))
-  (gr_text github.com/tebl (at 140.335 89.535) (layer F.SilkS)
+  (gr_text github.com/tebl (at 137.16 84.455) (layer F.SilkS)
     (effects (font (size 1 1) (thickness 0.15)))
   )
@@
     (effects (font (size 0.8 0.8) (thickness 0.15)) (justify left mirror))
   )
-  (gr_text "Commodore 64\nModulator Replacement\n(\"Longboard\" edition)" (at 140.97 84.455) (layer F.SilkS)
+  (gr_text "Commodore 64\nModulator Replacement\n(\"Longboard\" edition)" (at 137.16 79.375) (layer F.SilkS)
     (effects (font (size 1.5 1.5) (thickness 0.15)))
   )
@@
   (segment (start 135.89 109.855) (end 135.89 106.045) (width 0.5) (layer F.Cu) (net 6))
   (segment (start 138.515 121.4) (end 138.515 112.48) (width 0.5) (layer F.Cu) (net 6))
-  (segment (start 165.1 92.71) (end 167.64 92.71) (width 0.5) (layer F.Cu) (net 7))
-  (segment (start 175.895 83.82) (end 168.91 83.82) (width 0.5) (layer F.Cu) (net 7))
-  (segment (start 168.91 83.82) (end 167.64 85.09) (width 0.5) (layer F.Cu) (net 7))
-  (segment (start 167.64 85.09) (end 167.64 92.71) (width 0.5) (layer F.Cu) (net 7))
-  (segment (start 167.64 92.71) (end 167.64 94.615) (width 0.5) (layer F.Cu) (net 7))
-  (segment (start 175.895 76.835) (end 175.895 71.755) (width 0.5) (layer F.Cu) (net 7))
-  (segment (start 175.895 83.82) (end 175.895 76.835) (width 0.5) (layer F.Cu) (net 7))
+  (segment (start 167.64 94.615) (end 165.735 92.71) (width 0.5) (layer F.Cu) (net 7))
+  (segment (start 158.75 92.71) (end 154.94 92.71) (width 0.5) (layer F.Cu) (net 7))
   (segment (start 165.1 92.71) (end 158.75 92.71) (width 0.5) (layer F.Cu) (net 7))
-  (segment (start 158.75 92.71) (end 130.81 92.71) (width 0.5) (layer F.Cu) (net 7))
+  (segment (start 165.1 92.71) (end 165.735 92.71) (width 0.5) (layer F.Cu) (net 7))
+  (segment (start 154.94 90.17) (end 154.94 92.71) (width 0.5) (layer F.Cu) (net 7))
+  (segment (start 154.94 92.71) (end 130.81 92.71) (width 0.5) (layer F.Cu) (net 7))
   (segment (start 130.81 92.71) (end 130.175 93.345) (width 0.5) (layer F.Cu) (net 7))
   (segment (start 130.175 93.98) (end 130.175 97.79) (width 0.5) (layer F.Cu) (net 7))
   (segment (start 130.175 93.345) (end 130.175 93.98) (width 0.5) (layer F.Cu) (net 7))
-  (segment (start 167.64 94.615) (end 167.005 94.615) (width 0.5) (layer F.Cu) (net 7))
   (segment (start 123.19 97.79) (end 130.175 97.79) (width 0.5) (layer B.Cu) (net 7))
   (segment (start 130.175 97.79) (end 135.255 97.79) (width 0.5) (layer F.Cu) (net 7))
@@
   (segment (start 163.83 116.205) (end 165.035 117.41) (width 0.25) (layer F.Cu) (net 19))
   (segment (start 165.1 121.335) (end 165.035 121.4) (width 0.25) (layer F.Cu) (net 19))
+  (segment (start 175.895 83.82) (end 156.21 83.82) (width 0.5) (layer F.Cu) (net 20))
+  (segment (start 156.21 83.82) (end 154.94 82.55) (width 0.5) (layer F.Cu) (net 20))
+  (segment (start 175.895 76.835) (end 175.895 71.755) (width 0.5) (layer F.Cu) (net 20))
+  (segment (start 175.895 83.82) (end 175.895 76.835) (width 0.5) (layer F.Cu) (net 20))
   (zone (net 3) (net_name GND) (layer B.Cu) (hatch edge 0.508)
     (connect_pads (clearance 0.508))

Commit message: Updated PCB layout
Parts:
- added C8: 10uF, Capacitors_THT:CP_Radial_D5.0mm_P2.50mm, F.Cu at (153.7, 70.5)
- added C9: 10uF, Capacitors_THT:CP_Radial_D5.0mm_P2.50mm, F.Cu at (175.9, 70.5)
- C4: footprint Capacitors_THT:CP_Radial_D4.0mm_P2.00mm -> Capacitors_THT:CP_Radial_D5.0mm_P2.50mm
- J4: value AUD_STEREO -> AUD_RIGHT; footprint Pin_Headers:Pin_Header_Straight_1x01_Pitch2.54mm -> Pin_Headers:Pin_Header_Straight_1x02_Pitch2.54mm
- moved J4 33.8 mm to (153.7, 76.8), turned to 90 degrees
- moved C7 4.02 mm to (179.7, 73.0), turned to 90 degrees
- moved C5 2.62 mm to (178.4, 77.5), turned to 180 degrees
- moved C4 2.54 mm to (178.4, 95.2), turned to 180 degrees
- moved U1 2.54 mm to (178.4, 88.9)
- moved D1 1.91 mm to (156.8, 90.2)
Connections:
- J5 pad 2: /AUD_R -> Net-(C9-Pad2)
- J5 pad 5: AUDIO_IN -> Net-(C8-Pad2)
Routing:
- net Net-(J4-Pad1): track 82.0 -> 17.5 mm
- net AUDIO_IN: track 65.5 -> 72.6 mm, vias 3 -> 1
- net /AUD_R: track 9.41 -> 15.8 mm
- net Net-(C8-Pad2): track 0.00 -> 4.02 mm
- net Net-(C9-Pad2): track 0.00 -> 3.93 mm
- net +9V: track 37.5 -> 40.4 mm
- net Net-(C5-Pad1): track 33.5 -> 33.4 mm, vias 0 -> 2
Other:
- board text added: "L1, C8, C9, D1 pads can be shorted, C2 & C3 can be left out."
- board text added: "SID#2 IN"
- board text removed: "L1 & D1 pads can be shorted, C2 & C3 can be left out."
- board text removed: "Right ch. IN"
