File: C64 Modulator.kicad_pcb (KiCad board)
At the start: 2 copper layers, 63.5 x 63.4 mm, 42 parts, among them J10 , J11 , J12 , J13 , J14 , J2 8765, J3 4321, J4 AUD_RIGHT, J5 TRS_3.5mm, J6 RCA_PLUG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

Commit message: Removed C8/C9
Parts:
- removed C8, C9: 10uF, Capacitors_THT:CP_Radial_D5.0mm_P2.50mm
Connections:
- J5 pad 2: Net-(C9-Pad2) -> /AUD_R
- J5 pad 5: Net-(C8-Pad2) -> AUDIO_IN
Routing:
- net /AUD_R: track 15.8 -> 9.41 mm
- net AUDIO_IN: track 72.6 -> 66.4 mm
- net Net-(C8-Pad2): track 4.02 -> 0.00 mm
- net Net-(C9-Pad2): track 3.93 -> 0.00 mm
Other:
- board text added: "Revision C"
- board text removed: "Revision B"

Commit message: Updated gerbers
Other:
- board text added: "AUD"
Changed lines of the file:
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@@
     (links 62)
     (no_connects 0)
-    (area 113.03 50.092 185.683334 130.175001)
+    (area 118.669999 62.154999 182.360001 125.745001)
     (thickness 1.6)
-    (drawings 113)
+    (drawings 115)
     (tracks 150)
     (zones 0)
@@
     )
   )
+  (gr_text AUD (at 153.67 74.93 90) (layer F.SilkS)
+    (effects (font (size 1 1) (thickness 0.15)) (justify left))
+  )
+  (gr_text GND (at 156.21 74.93 90) (layer F.SilkS)
+    (effects (font (size 1 1) (thickness 0.15)) (justify left))
+  )
   (gr_text "SID#2 IN" (at 154.94 79.375) (layer F.SilkS)
     (effects (font (size 0.8 0.8) (thickness 0.15)))
@@
   (segment (start 167.64 113.665) (end 167.005 113.665) (width 0.25) (layer F.Cu) (net 12))
   (segment (start 153.67 113.665) (end 167.005 113.665) (width 0.25) (layer F.Cu) (net 12))
-  (segment (start 162.29 76.835) (end 160.655 76.835) (width 0.5) (layer F.Cu) (net 13) (status 400000))
-  (segment (start 159.83 76.01) (end 159.83 71.355) (width 0.5) (layer F.Cu) (net 13) (status 800000))
+  (segment (start 162.29 76.835) (end 160.655 76.835) (width 0.5) (layer F.Cu) (net 13))
+  (segment (start 159.83 76.01) (end 159.83 71.355) (width 0.5) (layer F.Cu) (net 13))
   (segment (start 160.655 76.835) (end 159.83 76.01) (width 0.5) (layer F.Cu) (net 13))
   (segment (start 170.815 85.09) (end 170.815 82.55) (width 0.5) (layer F.Cu) (net 13))
@@
   (segment (start 154.94 79.375) (end 166.37 79.375) (width 0.5) (layer B.Cu) (net 14))
   (segment (start 153.67 78.105) (end 154.94 79.375) (width 0.5) (layer B.Cu) (net 14))
-  (segment (start 169.83 71.355) (end 169.83 73.375) (width 0.5) (layer F.Cu) (net 15) (status 400000))
-  (segment (start 164.83 75.2) (end 164.83 76.835) (width 0.5) (layer F.Cu) (net 15) (status 800000))
+  (segment (start 169.83 71.355) (end 169.83 73.375) (width 0.5) (layer F.Cu) (net 15))
+  (segment (start 164.83 75.2) (end 164.83 76.835) (width 0.5) (layer F.Cu) (net 15))
   (segment (start 165.735 74.295) (end 164.83 75.2) (width 0.5) (layer F.Cu) (net 15))
   (segment (start 168.91 74.295) (end 165.735 74.295) (width 0.5) (layer F.Cu) (net 15))
