File: C64 Modulator.sch (KiCad schematic (older format))
At the start: 40 parts, among them J10 , J11 , J12 , J13 , J14 , J2 8765, J3 4321, J4 AUD_RIGHT, J5 TRS_3.5mm, J6 RCA_PLUG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

Commit message: Updated gerbers
Other:
- note added: "C"
- note removed: "B"
Changed lines of the file:
@@
 C64 Modulator replacement, "Longboard" edition
 Text Notes 10550 7650 0    60   ~ 0
-B
+C
 $EndSCHEMATC
